Commit message: updated urdf and build architecture for ros2 humble

File: taurob_tracker_description/urdf/tracker_standalone.urdf.xacro (robot description, xacro)
@@ -2,9 +2,8 @@
 <robot name="taurob_tracker"
     xmlns:xacro="http://playerstage.sourceforge.net/gazebo/xmlschema/#interface">
-    <property name="flipper_offset_x" value="0.205" />
-    <property name="flipper_offset_y" value="0.15" />
-    <property name="flipper_offset_z" value="0.099" />
-    <property name="M_PI" value="3.14159" />
-    <property name="angle_deg" value="45" />
+    <xacro:property name="flipper_offset_x" value="0.205" />
+    <xacro:property name="flipper_offset_y" value="0.15" />
+    <xacro:property name="flipper_offset_z" value="0.099" />
+    <xacro:property name="angle_deg" value="45" />
     <xacro:include filename="$(find taurob_tracker_description)/urdf/tracker_chassis.urdf.xacro.xml" />
     <xacro:tracker_chassis_macro />

File: taurob_tracker_description/urdf/tracker_with_arm.urdf.xacro (robot description, xacro)
@@ -2,17 +2,17 @@
 <robot name="taurob_tracker"
     xmlns:xacro="http://playerstage.sourceforge.net/gazebo/xmlschema/#interface">
-    <property name="flipper_offset_x" value="0.205" />
-    <property name="flipper_offset_y" value="0.15" />
-    <property name="flipper_offset_z" value="0.099" />
-    <property name="M_PI" value="3.14159" />
-    <property name="angle_deg" value="45" />
+    <xacro:property name="flipper_offset_x" value="0.205" />
+    <xacro:property name="flipper_offset_y" value="0.15" />
+    <xacro:property name="flipper_offset_z" value="0.099" />
+    <xacro:property name="angle_deg" value="45" />
+    <xacro:property name="mpi" value="3.141519" />
     <xacro:include filename="$(find taurob_tracker_description)/urdf/tracker_chassis.urdf.xacro.xml" />
-    <tracker_chassis_macro />
+    <xacro:tracker_chassis_macro />
     <!--Examples of adding additional robot parts below-->
     <xacro:include filename="$(find taurob_arm_description)/urdf/taurob_arm_collision_geoms_simple.urdf.xacro.xml" />
     <xacro:include filename="$(find taurob_arm_description)/urdf/taurob_arm_macros.urdf.xacro.xml" />
-    <taurob_arm_simple_eef_macro parent="base_link">
-      <origin xyz="0.12 0 0.185" rpy="0 0 ${M_PI/2}"/>
-    </taurob_arm_simple_eef_macro>
+    <xacro:taurob_arm_simple_eef_macro parent="chassis_link">
+      <origin xyz="0.0 0 0.0" rpy="0 0 ${mpi/2}"/>
+    </xacro:taurob_arm_simple_eef_macro>
     <!--
     <xacro:include filename="$(find hector_components_description)/urdf/spinning_hokuyo_utm30lx.urdf.xacro" />
