Commit message: added a diff drive controller and two wheels. next up, try it in the python agx scene builder and try to add tracks

File: taurob_agx_bringup/urdf/taurob.agx_ros2_control.xacro (robot description, xacro)
@@ -25,4 +25,18 @@
         <xacro:configure_joint joint_name="arm_joint_2" initial_position="0.0" min_vel="-2.0" max_vel="2.0"/>
         <xacro:configure_joint joint_name="arm_joint_3" initial_position="0.0" min_vel="-2.0" max_vel="2.0"/>
+        <xacro:macro name="configure_wheel" params="joint_name agx_name min_vel max_vel">
+          <joint name="${joint_name}">
+            <param name="agx_name">${agx_name}</param>
+            <param name="sign">1</param>
+            <command_interface name="velocity">
+              <param name="min">${min_vel}</param>
+              <param name="max">${max_vel}</param>
+            </command_interface>
+            <state_interface name="position"/>
+            <state_interface name="velocity"/>
+          </joint>
+        </xacro:macro>
+        <xacro:configure_wheel joint_name="left_wheel_joint" agx_name="left_wheel_joint" min_vel="-2.0" max_vel="2.0"/>
+        <xacro:configure_wheel joint_name="right_wheel_joint" agx_name="right_wheel_joint" min_vel="-2.0" max_vel="2.0"/>
     </ros2_control>
   </xacro:macro>

File: taurob_agx_bringup/urdf/tracker_chassis.urdf.xacro (robot description, xacro)
@@ -23,96 +23,96 @@
     </joint>
     <link name="flipper_link_1">
-      <xacro:inertial_cuboid_with_pose mass="1.0" x_length="${tracker_base_size_x*0.5}" y_length="${track_width*2}" z_length="0.17651" >
+      <xacro:inertial_cuboid_with_pose mass="1.0" x_length="${tracker_base_size_x*0.5}" y_length="${track_width/2}" z_length="0.017651" >
         <origin xyz="${tracker_base_size_x*0.5-track_wheel_radius*2} 0.0 0.0" rpy="0 0 0" />
       </xacro:inertial_cuboid_with_pose>
       <origin xyz="0 0 0" rpy="0 0 0" />
       <visual>
-        <origin xyz="${tracker_base_size_x*0.5-track_wheel_radius+flipper_offset_x} -${track_offset_y} 0.0" rpy="${pi/2} 0 0"/>
+        <origin xyz="${tracker_base_size_x*0.5-track_wheel_radius+flipper_offset_x} -${track_offset_y+track_width/2} 0.0" rpy="${pi/2} 0 0"/>
         <geometry>
-          <cylinder length="${track_width}" radius="${track_wheel_radius}"/>
+          <cylinder length="${track_width/2}" radius="${track_wheel_radius/2}"/>
         </geometry>
         <material name="black">
-          <color rgba="0 0 0 1"/>
+          <color rgba="0.8 0.8 0.8 1"/>
         </material>
       </visual>
       <visual>
-        <origin xyz="0 -${track_offset_y} 0.0" rpy="${pi/2} 0 0"/>
+        <origin xyz="0 -${track_offset_y+track_width/2} 0.0" rpy="${pi/2} 0 0"/>
         <geometry>
-          <cylinder length="${track_width}" radius="${track_wheel_radius}"/>
+          <cylinder length="${track_width/2}" radius="${track_wheel_radius/2}"/>
         </geometry>
         <material name="black">
-          <color rgba="0 0 0 1"/>
+          <color rgba="0.8 0.8 0.8 1"/>
         </material>
       </visual>
       <visual>
-        <origin xyz="${(tracker_base_size_x*0.5-track_wheel_radius+flipper_offset_x)*0.5} -${track_offset_y} 0.0" rpy="0 0 0"/>
+        <origin xyz="${(tracker_base_size_x*0.5-track_wheel_radius+flipper_offset_x)*0.5} -${track_offset_y+track_width/2} 0.0" rpy="0 0 0"/>
         <geometry>
-          <box size="${tracker_base_size_x*0.5-track_wheel_radius+flipper_offset_x} ${track_width} ${track_wheel_radius*2}"/>
+          <box size="${tracker_base_size_x*0.5-track_wheel_radius+flipper_offset_x} ${track_width/2} ${track_wheel_radius}"/>
         </geometry>
         <material name="black">
-          <color rgba="0 0 0 1"/>
+          <color rgba="0.8 0.8 0.8 1"/>
         </material>
       </visual>
       <visual>
-        <origin xyz="${tracker_base_size_x*0.5-track_wheel_radius+flipper_offset_x} ${track_offset_y} 0.0" rpy="${pi/2} 0 0"/>
+        <origin xyz="${tracker_base_size_x*0.5-track_wheel_radius+flipper_offset_x} ${track_offset_y+track_width/2} 0.0" rpy="${pi/2} 0 0"/>
         <geometry>
-          <cylinder length="${track_width}" radius="${track_wheel_radius}"/>
+          <cylinder length="${track_width/2}" radius="${track_wheel_radius/2}"/>
         </geometry>
         <material name="black">
-          <color rgba="0 0 0 1"/>
+          <color rgba="0.8 0.8 0.8 1"/>
         </material>
       </visual>
       <visual>
-        <origin xyz="0 ${track_offset_y} 0.0" rpy="${pi/2} 0 0"/>
+        <origin xyz="0 ${track_offset_y+track_width/2} 0.0" rpy="${pi/2} 0 0"/>
         <geometry>
-          <cylinder length="${track_width}" radius="${track_wheel_radius}"/>
+          <cylinder length="${track_width/2}" radius="${track_wheel_radius/2}"/>
         </geometry>
         <material name="black">
-          <color rgba="0 0 0 1"/>
+          <color rgba="0.8 0.8 0.8 1"/>
         </material>
       </visual>
       <visual>
-        <origin xyz="${(tracker_base_size_x*0.5-track_wheel_radius+flipper_offset_x)*0.5} ${track_offset_y} 0.0" rpy="0 0 0"/>
+        <origin xyz="${(tracker_base_size_x*0.5-track_wheel_radius+flipper_offset_x)*0.5} ${track_offset_y+track_width/2} 0.0" rpy="0 0 0"/>
         <geometry>
-          <box size="${tracker_base_size_x*0.5-track_wheel_radius+flipper_offset_x} ${track_width} ${track_wheel_radius*2}"/>
+          <box size="${tracker_base_size_x*0.5-track_wheel_radius+flipper_offset_x} ${track_width/2} ${track_wheel_radius}"/>
         </geometry>
         <material name="black">
-          <color rgba="0 0 0 1"/>
+          <color rgba="0.8 0.8 0.8 1"/>
         </material>
       </visual>
       <collision>
-        <origin xyz="${tracker_base_size_x*0.5-track_wheel_radius+flipper_offset_x} -${track_offset_y} 0.0" rpy="${pi/2} 0 0"/>
+        <origin xyz="${tracker_base_size_x*0.5-track_wheel_radius+flipper_offset_x} -${track_offset_y+track_width/2} 0.0" rpy="${pi/2} 0 0"/>
         <geometry>
-          <cylinder length="${track_width}" radius="${track_wheel_radius}"/>
+          <cylinder length="${track_width/2}" radius="${track_wheel_radius/2}"/>
         </geometry>
       </collision>
       <collision>
-        <origin xyz="0 -${track_offset_y} 0.0" rpy="${pi/2} 0 0"/>
+        <origin xyz="0 -${track_offset_y+track_width/2} 0.0" rpy="${pi/2} 0 0"/>
         <geometry>
-          <cylinder length="${track_width}" radius="${track_wheel_radius}"/>
+          <cylinder length="${track_width/2}" radius="${track_wheel_radius/2}"/>
         </geometry>
       </collision>
       <collision>
-        <origin xyz="${(tracker_base_size_x*0.5-track_wheel_radius+flipper_offset_x)*0.5} -${track_offset_y} 0.0" rpy="0 0 0"/>
+        <origin xyz="${(tracker_base_size_x*0.5-track_wheel_radius+flipper_offset_x)*0.5} -${track_offset_y+track_width/2} 0.0" rpy="0 0 0"/>
         <geometry>
-          <box size="${tracker_base_size_x*0.5-track_wheel_radius+flipper_offset_x} ${track_width} ${track_wheel_radius*2}"/>
+          <box size="${tracker_base_size_x*0.5-track_wheel_radius+flipper_offset_x} ${track_width/2} ${track_wheel_radius}"/>
         </geometry>
       </collision>
       <collision>
-        <origin xyz="${tracker_base_size_x*0.5-track_wheel_radius+flipper_offset_x} ${track_offset_y} 0.0" rpy="${pi/2} 0 0"/>
+        <origin xyz="${tracker_base_size_x*0.5-track_wheel_radius+flipper_offset_x} ${track_offset_y+track_width/2} 0.0" rpy="${pi/2} 0 0"/>
         <geometry>
-          <cylinder length="${track_width}" radius="${track_wheel_radius}"/>
+          <cylinder length="${track_width/2}" radius="${track_wheel_radius/2}"/>
         </geometry>
       </collision>
       <collision>
-        <origin xyz="0 ${track_offset_y} 0.0" rpy="${pi/2} 0 0"/>
+        <origin xyz="0 ${track_offset_y+track_width/2} 0.0" rpy="${pi/2} 0 0"/>
         <geometry>
-          <cylinder length="${track_width}" radius="${track_wheel_radius}"/>
+          <cylinder length="${track_width/2}" radius="${track_wheel_radius/2}"/>
         </geometry>
       </collision>
       <collision>
-        <origin xyz="${(tracker_base_size_x*0.5-track_wheel_radius+flipper_offset_x)*0.5} ${track_offset_y} 0.0" rpy="0 0 0"/>
+        <origin xyz="${(tracker_base_size_x*0.5-track_wheel_radius+flipper_offset_x)*0.5} ${track_offset_y+track_width/2} 0.0" rpy="0 0 0"/>
         <geometry>
-          <box size="${tracker_base_size_x*0.5-track_wheel_radius+flipper_offset_x} ${track_width} ${track_wheel_radius*2}"/>
+          <box size="${tracker_base_size_x*0.5-track_wheel_radius+flipper_offset_x} ${track_width/2} ${track_wheel_radius}"/>
         </geometry>
       </collision>
@@ -143,10 +143,57 @@
       <!--Chassis middle-->
       <collision>
-        <origin xyz="${tracker_base_offset_x-0.13} 0.0 ${tracker_base_offset_z+0.005}" rpy="0 0 0"/>
+        <origin xyz="0.0 0.0 0.0" rpy="0 0 0" />
         <geometry>
-          <box size="0.7 0.5 0.15"/>
+          <mesh filename="package://taurob_agx_bringup/meshes/tracker_chassis_no_tracks.dae"/>
         </geometry>
       </collision>
     </link>
+    <!-- active wheels -->
+    <link name="left_wheel">
+      <visual>
+        <origin xyz="0.0 0.0 0.0" rpy="${pi/2} 0 0"/>
+        <geometry>
+          <cylinder length="${track_width/2}" radius="${track_wheel_radius}"/>
+        </geometry>
+        <material name="wheel_black">
+          <color rgba="0 0 0 1"/>
+        </material>
+      </visual>
+      <collision>
+        <origin xyz="0.0 0.0 0.0" rpy="${pi/2} 0 0"/>
+        <geometry>
+          <cylinder length="${track_width/2}" radius="${track_wheel_radius}"/>
+        </geometry>
+      </collision>
+    </link>
+    <joint name="left_wheel_joint" type="continuous">
+      <origin xyz="${tracker_base_offset_x-flipper_offset_x} ${track_offset_y-0.01} ${track_offset_z}" rpy="0 0 0" />
+      <axis xyz="0 1 0"/>
+      <parent link="chassis_link"/>
+      <child link="left_wheel"/>
+    </joint>
+    <link name="right_wheel">
+      <visual>
+        <origin xyz="0.0 0.0 0.0" rpy="${pi/2} 0 0"/>
+        <geometry>
+          <cylinder length="${track_width/2}" radius="${track_wheel_radius}"/>
+        </geometry>
+        <material name="wheel_black">
+          <color rgba="0 0 0 1"/>
+        </material>
+      </visual>
+      <collision>
+        <origin xyz="0.0 0.0 0.0" rpy="${pi/2} 0 0"/>
+        <geometry>
+          <cylinder length="${track_width/2}" radius="${track_wheel_radius}"/>
+        </geometry>
+      </collision>
+    </link>
+    <joint name="right_wheel_joint" type="continuous">
+      <origin xyz="${tracker_base_offset_x-flipper_offset_x} -${track_offset_y-0.01} ${track_offset_z}" rpy="0 0 0" />
+      <axis xyz="0 1 0"/>
+      <parent link="chassis_link"/>
+      <child link="right_wheel"/>
+    </joint>
   </xacro:macro>
 </robot>
